File: gateway.sch (EAGLE design)
At the start: 71 parts, among them IC2 24AA00OT, J1 MAGJACK, Q3 BC817, U3 TPD4E002DRLR, U5 TPD4E002DRLR, U6 TPD4E002DRLR, U7 TPD4E002DRLR, Y2 16MHz

Commit message: Version 5
Parts:
- added U8: 74LVC1G04GW, 74LVC1G04GW_inverter:74LVC1G04GW
Connections:
- new net ETH_50MHZ_180_OUT: U$62.NINT/REFCLKO, U8.A
- net 3.3V: now also U8.VCC
- net ETH_50MHZ: now also U8.Y; no longer U$62.NINT/REFCLKO
- net GND: now also U8.GND
Other:
- note added: "Inverter needed for 180° phase shift"
- note added: "as SMSC PHY output not RMII compliant"
- moved on the sheet: CN2
Changed lines of the file:
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@@
 <?xml version="1.0" encoding="utf-8"?>
 <!DOCTYPE eagle SYSTEM "eagle.dtd">
-<eagle version="6.2">
+<eagle version="6.4">
 <drawing>
 <settings>
@@
 <part name="U$34" library="microbuilder" deviceset="GND" device=""/>
 <part name="C26" library="resistor" deviceset="C-EU" device="C0603K" value="470pF"/>
+<part name="U$19" library="microbuilder" deviceset="3.3V" device=""/>
+<part name="U$20" library="microbuilder" deviceset="GND" device=""/>
+<part name="U8" library="74LVC1G04GW_inverter" deviceset="74LVC1G04GW" device=""/>
+<part name="FRAME3" library="SparkFun" deviceset="FRAME-LETTER" device=""/>
 </parts>
 <sheets>
@@
 <plain>
 <text x="292.1" y="175.26" size="1.778" layer="97">TODO: Switch power supply for SD</text>
+<text x="414.02" y="38.1" size="2.54" layer="97" font="vector">Inverter needed for 180° phase shift</text>
+<text x="414.02" y="33.02" size="2.54" layer="97" font="vector">as SMSC PHY output not RMII compliant</text>
 </plain>
 <instances>
@@
 <instance part="U$56" gate="G$1" x="317.5" y="45.72"/>
 <instance part="U$57" gate="G$1" x="317.5" y="76.2"/>
-<instance part="U$59" gate="G$1" x="309.88" y="114.3" rot="MR0"/>
+<instance part="U$59" gate="G$1" x="302.26" y="116.84" rot="MR0"/>
 <instance part="X1" gate="G$1" x="739.14" y="170.18"/>
 <instance part="U$2" gate="G$1" x="695.96" y="223.52"/>
@@
 <instance part="U$74" gate="P1" x="45.72" y="83.82" rot="R180"/>
 <instance part="U$76" gate="G$1" x="53.34" y="78.74"/>
-<instance part="U$79" gate="G$1" x="297.18" y="139.7" rot="MR0"/>
+<instance part="U$79" gate="G$1" x="289.56" y="142.24" rot="MR0"/>
 <instance part="R14" gate="G$1" x="657.86" y="81.28"/>
 <instance part="R15" gate="G$1" x="657.86" y="96.52"/>
@@
 <instance part="C3" gate="G$1" x="215.9" y="139.7"/>
 <instance part="U$73" gate="G$1" x="215.9" y="129.54"/>
-<instance part="CN2" gate="G$1" x="320.04" y="147.32"/>
-<instance part="U$81" gate="G$1" x="312.42" y="114.3" rot="MR0"/>
-<instance part="U$95" gate="G$1" x="297.18" y="114.3" rot="MR0"/>
+<instance part="CN2" gate="G$1" x="312.42" y="149.86"/>
+<instance part="U$81" gate="G$1" x="304.8" y="116.84" rot="MR0"/>
+<instance part="U$95" gate="G$1" x="289.56" y="116.84" rot="MR0"/>
 <instance part="C15" gate="G$1" x="492.76" y="109.22" rot="R180"/>
 <instance part="R11" gate="G$1" x="335.28" y="88.9" rot="R180"/>
@@
 <instance part="U$34" gate="G$1" x="541.02" y="104.14"/>
 <instance part="C26" gate="G$1" x="541.02" y="111.76"/>
+<instance part="U$19" gate="G$1" x="462.28" y="73.66"/>
+<instance part="U$20" gate="G$1" x="462.28" y="48.26"/>
+<instance part="U8" gate="A" x="441.96" y="63.5" rot="MR0"/>
+<instance part="FRAME3" gate="G$2" x="215.9" y="-27.94"/>
 </instances>
 <busses>
@@
 </segment>
 <segment>
-<wire x1="309.88" y1="116.84" x2="309.88" y2="119.38" width="0.1524" layer="91"/>
+<wire x1="302.26" y1="119.38" x2="302.26" y2="121.92" width="0.1524" layer="91"/>
 <pinref part="U$59" gate="G$1" pin="GND"/>
 <pinref part="CN2" gate="G$1" pin="GND2"/>
 </segment>
 <segment>
-<wire x1="312.42" y1="116.84" x2="312.42" y2="119.38" width="0.1524" layer="91"/>
+<wire x1="304.8" y1="119.38" x2="304.8" y2="121.92" width="0.1524" layer="91"/>
 <pinref part="U$81" gate="G$1" pin="GND"/>
 <pinref part="CN2" gate="G$1" pin="GND3"/>
 </segment>
 <segment>
-<wire x1="297.18" y1="116.84" x2="297.18" y2="127" width="0.1524" layer="91"/>
-<wire x1="304.8" y1="127" x2="297.18" y2="127" width="0.1524" layer="91"/>
-<wire x1="304.8" y1="129.54" x2="297.18" y2="129.54" width="0.1524" layer="91"/>
-<wire x1="297.18" y1="129.54" x2="297.18" y2="127" width="0.1524" layer="91"/>
-<wire x1="304.8" y1="134.62" x2="297.18" y2="134.62" width="0.1524" layer="91"/>
-<wire x1="297.18" y1="134.62" x2="297.18" y2="129.54" width="0.1524" layer="91"/>
-<junction x="297.18" y="129.54"/>
-<junction x="297.18" y="127"/>
+<wire x1="289.56" y1="119.38" x2="289.56" y2="129.54" width="0.1524" layer="91"/>
+<wire x1="297.18" y1="129.54" x2="289.56" y2="129.54" width="0.1524" layer="91"/>
+<wire x1="297.18" y1="132.08" x2="289.56" y2="132.08" width="0.1524" layer="91"/>
+<wire x1="289.56" y1="132.08" x2="289.56" y2="129.54" width="0.1524" layer="91"/>
+<wire x1="297.18" y1="137.16" x2="289.56" y2="137.16" width="0.1524" layer="91"/>
+<wire x1="289.56" y1="137.16" x2="289.56" y2="132.08" width="0.1524" layer="91"/>
+<junction x="289.56" y="132.08"/>
+<junction x="289.56" y="129.54"/>
 <pinref part="U$95" gate="G$1" pin="GND"/>
 <pinref part="CN2" gate="G$1" pin="GND"/>
@@
 <pinref part="U$34" gate="G$1" pin="GND"/>
 <pinref part="C26" gate="G$1" pin="2"/>
+</segment>
+<segment>
+<pinref part="U$20" gate="G$1" pin="GND"/>
+<wire x1="462.28" y1="53.34" x2="462.28" y2="50.8" width="0.1524" layer="91"/>
+<pinref part="U8" gate="A" pin="GND"/>
+<wire x1="459.74" y1="53.34" x2="462.28" y2="53.34" width="0.1524" layer="91"/>
 </segment>
 </net>
@@
 </segment>
 <segment>
-<wire x1="297.18" y1="139.7" x2="297.18" y2="137.16" width="0.1524" layer="91"/>
-<wire x1="297.18" y1="137.16" x2="304.8" y2="137.16" width="0.1524" layer="91"/>
+<wire x1="289.56" y1="142.24" x2="289.56" y2="139.7" width="0.1524" layer="91"/>
+<wire x1="289.56" y1="139.7" x2="297.18" y2="139.7" width="0.1524" layer="91"/>
 <pinref part="U$79" gate="G$1" pin="3.3V"/>
 <pinref part="CN2" gate="G$1" pin="VDD"/>
@@
 <junction x="485.14" y="116.84"/>
 </segment>
+<segment>
+<pinref part="U$19" gate="G$1" pin="3.3V"/>
+<wire x1="462.28" y1="68.58" x2="462.28" y2="73.66" width="0.1524" layer="91"/>
+<pinref part="U8" gate="A" pin="VCC"/>
+<wire x1="459.74" y1="68.58" x2="462.28" y2="68.58" width="0.1524" layer="91"/>
+</segment>
 </net>
 <net name="TD-" class="0">
@@
 </segment>
 <segment>
-<pinref part="U$62" gate="G$1" pin="NINT/REFCLKO"/>
-<wire x1="487.68" y1="63.5" x2="467.36" y2="63.5" width="0.1524" layer="91"/>
-<label x="469.9" y="63.5" size="1.778" layer="95"/>
+<wire x1="424.18" y1="68.58" x2="406.4" y2="68.58" width="0.1524" layer="91"/>
+<label x="408.94" y="68.58" size="1.778" layer="95"/>
+<pinref part="U8" gate="A" pin="Y"/>
 </segment>
 </net>
@@
 <net name="SD_CLK" class="0">
 <segment>
-<wire x1="304.8" y1="149.86" x2="281.94" y2="149.86" width="0.1524" layer="91"/>
-<label x="294.64" y="149.86" size="1.778" layer="95" rot="MR0"/>
+<wire x1="297.18" y1="152.4" x2="274.32" y2="152.4" width="0.1524" layer="91"/>
+<label x="287.02" y="152.4" size="1.778" layer="95" rot="MR0"/>
 <pinref part="CN2" gate="G$1" pin="SCLK"/>
 </segment>
@@
 <net name="SD_MOSI" class="0">
 <segment>
-<wire x1="304.8" y1="152.4" x2="281.94" y2="152.4" width="0.1524" layer="91"/>
-<label x="294.64" y="152.4" size="1.778" layer="95" rot="MR0"/>
+<wire x1="297.18" y1="154.94" x2="274.32" y2="154.94" width="0.1524" layer="91"/>
+<label x="287.02" y="154.94" size="1.778" layer="95" rot="MR0"/>
 <pinref part="CN2" gate="G$1" pin="DATA_IN"/>
 </segment>
@@
 <net name="SD_CS" class="0">
 <segment>
-<wire x1="304.8" y1="147.32" x2="281.94" y2="147.32" width="0.1524" layer="91"/>
-<label x="294.64" y="147.32" size="1.778" layer="95" rot="MR0"/>
+<wire x1="297.18" y1="149.86" x2="274.32" y2="149.86" width="0.1524" layer="91"/>
+<label x="287.02" y="149.86" size="1.778" layer="95" rot="MR0"/>
 <pinref part="CN2" gate="G$1" pin="CS"/>
 </segment>
@@
 <net name="SD_MISO" class="0">
 <segment>
-<wire x1="304.8" y1="154.94" x2="281.94" y2="154.94" width="0.1524" layer="91"/>
-<label x="294.64" y="154.94" size="1.778" layer="95" rot="MR0"/>
+<wire x1="297.18" y1="157.48" x2="274.32" y2="157.48" width="0.1524" layer="91"/>
+<label x="287.02" y="157.48" size="1.778" layer="95" rot="MR0"/>
 <pinref part="CN2" gate="G$1" pin="DATA_OUT"/>
 </segment>
@@
 </segment>
 </net>
+<net name="ETH_50MHZ_180_OUT" class="0">
+<segment>
+<pinref part="U$62" gate="G$1" pin="NINT/REFCLKO"/>
+<wire x1="459.74" y1="63.5" x2="487.68" y2="63.5" width="0.1524" layer="91"/>
+<label x="464.82" y="63.5" size="1.778" layer="95"/>
+<pinref part="U8" gate="A" pin="A"/>
+</segment>
+</net>

Commit message: Version 6
Parts:
- removed C26: 470pF, resistor:C-EUC0603K
- removed C27: 100pF, resistor:C-EUC0603K
- removed C32: 10nF, resistor:C-EUC0603K
- removed C7: 100nF, resistor:C-EUC0603K
- removed CN1: (no value), microbuilder:DCBARREL
- removed Q2: (no value), microbuilder:MOSFET-P
- removed Q3: BC817, microbuilder:TRANSISTOR_NPN
- removed R10: 100K, microbuilder:RESISTOR0603MINI
- removed R11: 2.2K, microbuilder:RESISTOR0603MINI
- removed R2, R3, R4, R5: 49.9R, microbuilder:RESISTOR0603MINI
- removed U$74: SM04B-SURS-TF, con-jst:SM04B-SURS-TF
- removed U3, U5, U6, U7: TPD4E002DRLR, TPD4E002:TPD4E002DRLR
- removed X1: (no value), microbuilder:SMACONNECTOR
- added C5: 100nF, resistor:C-EUC1206
- added FB2: (no value), microbuilder:FERRITE
- added J$1: SMA_EDGE, SparkFun-Connectors:SMA_EDGE
- added JTAG1: (no value), microbuilder_v3:JTAG-CORTEXM3
- added R17, R21, R22, R6: 49.9R, microbuilder:RESISTOR0603MINI
- added U$18: J3011TIGHT, J3011:J3011TIGHT
- C4: device resistor:C-EUC0603K -> resistor:C-EUC1206
- C6: value 100nF -> 470pF
- J1: value MAGJACK -> POWER_JACKSMD_2; device SparkFun:MAGJACK -> SparkFun:POWER_JACKSMD_2
Connections:
- removed net N$6: U1.P0[10]/TXD2/SDA2/MAT3[0]
- removed net N$7: U1.P0[11]/RXD2/SCL2/MAT3[1]
- removed net PWR_MON_EN: R11.2, U1.P0[24]/AD0[1]/I2SRX_WS/CAP3[1]
- removed net PWR_MON_EN_SW: C27.1, Q2.G, Q3.C, R10.1
- removed net PWR_MON_SW: Q2.D, R9.2
- removed net Q3RES: Q3.B, R11.1
- removed net SD_EN: U1.P0[23]/AD0[0]/I2SRX_CLK/CAP3[0]
- new net CGND: FB2.P$2, U$18.SHIELD@0, U$18.SHIELD@1
- new net TDI: JTAG1.8, U1.TDI
- new net TDO_SWO: JTAG1.6, U1.TDO/SWO
- net !RESET!: now also JTAG1.10; no longer U$744.1
- net 3.3V: now also C5.1, JTAG1.1, R17.1, R21.1, R22.2, R6.2, U$18.RCT, U$18.TCT; no longer C26.1, C32.2, C7.1, J1.RCT, J1.TCT, R2.1, R3.2, R4.1, R5.2, U6.IO3, U6.IO4, U7.IO3, U7.IO4
- net GLED: now also U$18.GLED-, U1.P2[0]/PWM1[1]/TXD1; no longer J1.GLED-, U1.P2[3]/PWM1[4]/DCD1/TRACEDATA[2]
- net GLED+: now also U$18.GLED+; no longer J1.GLED+
- net GND: now also C5.2, FB2.P$1, J$1.GND@0, J$1.GND@1, J$1.GND@2, J$1.GND@3, J1.GND, J1.GNDBREAK, JTAG1.3, JTAG1.5, JTAG1.9, U$18.GND; no longer C26.2, C32.1, C7.2, CN1.GND, CN1.GNDBREAK, Q3.E, U$743.1, U$74P1.1, U$74P2.1, U3.GND, U5.GND, U5.IO1, U5.IO2, U6.GND, U7.GND, X1.GND1, X1.GND2, X1.GND3, X1.GND4
- net PWR: now also J1.PWR; no longer CN1.PWR, U5.IO3, U5.IO4
- net RADIORST: now also U1.P2[1]/PWM1[2]/RXD1; no longer U1.P2[5]/PWM1[6]/DTR1/TRACEDATA[0]
- net RD+: now also R21.2, U$18.RD+, U$62.TXP; no longer J1.RD+, R4.2, U$62.RXP, U6.IO2
- net RD-: now also R22.1, U$18.RD-, U$62.TXN; no longer J1.RD-, R5.1, U$62.RXN, U6.IO1
- net RPWR: now also R9.2; no longer C27.2, Q2.S, R10.2
- net SD_CLK: no longer U3.IO1
- net SD_CS: no longer U3.IO3
- net SD_MISO: no longer U3.IO2
- net SD_MOSI: no longer U3.IO4
- net SLP_TR: now also U1.P2[2]/PWM1[3]/CTS1/TRACEDATA[3]; no longer U1.P2[6]/PCAP1[0]/RI1/TRACECLK
- net TCK_SWDCLK: now also JTAG1.4; no longer U$741.1
- net TD+: now also R17.2, U$18.TD+, U$62.RXP; no longer J1.TD+, R2.2, U$62.TXP, U7.IO1
- net TD-: now also R6.1, U$18.TD-, U$62.RXN; no longer J1.TD-, R3.1, U$62.TXN, U7.IO2
- net TMS_SWDIO: now also JTAG1.2; no longer U$742.1
- net UNBAL: now also J$1.SIGNAL; no longer X1.ANT
- net YLED: now also U$18.YLED-, U1.P2[3]/PWM1[4]/DCD1/TRACEDATA[2]; no longer J1.YLED-, U1.P2[4]/PWM1[5]/DSR1/TRACEDATA[1]
- net YLED+: now also U$18.YLED+; no longer J1.YLED+
Other:
- note added: "Auto-MIDX means Rx/Tx swap is fine"
- note added: "as SMSC PHY output not RMII compliant!"
- note removed: "as SMSC PHY output not RMII compliant"
- moved on the sheet: C16, C23, C24, C25, C4, C6, IC1, Q1, R12, R13, R14, R15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
